File: hw/sch_pcb/QFHMIX01C.kicad_pcb (KiCad board)
At the start: 2 copper layers, 90.9 x 90.9 mm, 183 parts, among them J1 +9V, J2 HEADER_1x08, M1 HOLE, M2 HOLE, M3 HOLE, M4 HOLE, M5 HOLE, M6 HOLE, M7 HOLE, M8 HOLE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

Commit message: Generating manufacturing outputs.
Other:
- net class Default removed
