File: hw/sch_pcb/Power.kicad_sch (KiCad schematic)
At the start: 36 parts, among them U10 TPS563249, U11 TPS563249

Commit message: Oprava PCB.
Parts:
- C69, C70, C71, C72: footprint Mlab_C:SMD-0603 -> Capacitor_SMD:C_0603_1608Metric; UST_ID 5c70984712875079b91f8b4c -> (none)
- C81, C82: footprint Mlab_C:SMD-0603 -> Capacitor_SMD:C_0603_1608Metric; UST_ID 5c70984812875079b91f8bbe -> (none)
- R43, R44, R45, R46, R47, R48, R49, R50, R51, R52, R53, R54: footprint Mlab_R:SMD-0805 -> Resistor_SMD:R_0603_1608Metric
Changed lines of the file:
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@@
     (property "Reference" "R43" (id 0) (at 95.885 29.845 90))
     (property "Value" "100k" (id 1) (at 98.425 33.655 90))
-    (property "Footprint" "Mlab_R:SMD-0805" (id 2) (at 100.203 33.655 90)
+    (property "Footprint" "Resistor_SMD:R_0603_1608Metric" (id 2) (at 100.203 33.655 90)
       (effects (font (size 1.27 1.27)) hide)
     )
@@
     (property "Reference" "R44" (id 0) (at 95.885 41.91 90))
     (property "Value" "-" (id 1) (at 98.425 45.72 90))
-    (property "Footprint" "Mlab_R:SMD-0805" (id 2) (at 100.203 45.72 90)
+    (property "Footprint" "Resistor_SMD:R_0603_1608Metric" (id 2) (at 100.203 45.72 90)
       (effects (font (size 1.27 1.27)) hide)
     )
@@
     (property "Reference" "R45" (id 0) (at 96.52 78.105 90))
     (property "Value" "100k" (id 1) (at 99.06 81.915 90))
-    (property "Footprint" "Mlab_R:SMD-0805" (id 2) (at 100.838 81.915 90)
+    (property "Footprint" "Resistor_SMD:R_0603_1608Metric" (id 2) (at 100.838 81.915 90)
       (effects (font (size 1.27 1.27)) hide)
     )
@@
     (property "Reference" "R46" (id 0) (at 96.52 90.17 90))
     (property "Value" "-" (id 1) (at 99.06 93.98 90))
-    (property "Footprint" "Mlab_R:SMD-0805" (id 2) (at 100.838 93.98 90)
+    (property "Footprint" "Resistor_SMD:R_0603_1608Metric" (id 2) (at 100.838 93.98 90)
       (effects (font (size 1.27 1.27)) hide)
     )
@@
     (property "Reference" "R47" (id 0) (at 125.73 46.99 90))
     (property "Value" "10k" (id 1) (at 128.27 45.72 90))
-    (property "Footprint" "Mlab_R:SMD-0805" (id 2) (at 130.048 45.72 90)
+    (property "Footprint" "Resistor_SMD:R_0603_1608Metric" (id 2) (at 130.048 45.72 90)
       (effects (font (size 1.27 1.27)) hide)
     )
@@
     (property "Reference" "R48" (id 0) (at 126.365 95.25 90))
     (property "Value" "10k" (id 1) (at 128.905 93.98 90))
-    (property "Footprint" "Mlab_R:SMD-0805" (id 2) (at 130.683 93.98 90)
+    (property "Footprint" "Resistor_SMD:R_0603_1608Metric" (id 2) (at 130.683 93.98 90)
       (effects (font (size 1.27 1.27)) hide)
     )
@@
     (property "Reference" "R49" (id 0) (at 130.81 31.75 90))
     (property "Value" "0R" (id 1) (at 130.81 29.21 90))
-    (property "Footprint" "Mlab_R:SMD-0805" (id 2) (at 130.81 27.432 90)
+    (property "Footprint" "Resistor_SMD:R_0603_1608Metric" (id 2) (at 130.81 27.432 90)
       (effects (font (size 1.27 1.27)) hide)
     )
@@
     (property "Reference" "R50" (id 0) (at 131.445 80.01 90))
     (property "Value" "0R" (id 1) (at 131.445 77.47 90))
-    (property "Footprint" "Mlab_R:SMD-0805" (id 2) (at 131.445 75.692 90)
+    (property "Footprint" "Resistor_SMD:R_0603_1608Metric" (id 2) (at 131.445 75.692 90)
       (effects (font (size 1.27 1.27)) hide)
     )
@@
     (property "Reference" "R51" (id 0) (at 134.62 43.18 90))
     (property "Value" "45k3" (id 1) (at 135.89 40.64 90))
-    (property "Footprint" "Mlab_R:SMD-0805" (id 2) (at 135.89 38.862 90)
+    (property "Footprint" "Resistor_SMD:R_0603_1608Metric" (id 2) (at 135.89 38.862 90)
       (effects (font (size 1.27 1.27)) hide)
     )
@@
     (property "Reference" "R52" (id 0) (at 135.255 91.44 90))
     (property "Value" "73k2" (id 1) (at 136.525 88.9 90))
-    (property "Footprint" "Mlab_R:SMD-0805" (id 2) (at 136.525 87.122 90)
+    (property "Footprint" "Resistor_SMD:R_0603_1608Metric" (id 2) (at 136.525 87.122 90)
       (effects (font (size 1.27 1.27)) hide)
     )
@@
       (effects (font (size 1.27 1.27)) (justify left))
     )
-    (property "Footprint" "Mlab_R:SMD-0805" (id 2) (at 217.297 36.83 90)
+    (property "Footprint" "Resistor_SMD:R_0603_1608Metric" (id 2) (at 217.297 36.83 90)
       (effects (font (size 1.27 1.27)) hide)
     )
@@
       (effects (font (size 1.27 1.27)) (justify left))
     )
-    (property "Footprint" "Mlab_R:SMD-0805" (id 2) (at 217.297 85.09 90)
+    (property "Footprint" "Resistor_SMD:R_0603_1608Metric" (id 2) (at 217.297 85.09 90)
       (effects (font (size 1.27 1.27)) hide)
     )
@@
     (property "Reference" "C69" (id 0) (at 86.36 30.48 90))
     (property "Value" "100nF" (id 1) (at 88.9 39.37 90))
-    (property "Footprint" "Mlab_C:SMD-0603" (id 2) (at 84.1248 31.75 0)
-      (effects (font (size 1.27 1.27)) hide)
-    )
-    (property "Datasheet" "~" (id 3) (at 85.09 35.56 0)
-      (effects (font (size 1.27 1.27)) hide)
-    )
-    (property "UST_ID" "5c70984712875079b91f8b4c" (id 4) (at 85.09 35.56 0)
+    (property "Footprint" "Capacitor_SMD:C_0603_1608Metric" (id 2) (at 84.1248 31.75 0)
+      (effects (font (size 1.27 1.27)) hide)
+    )
+    (property "Datasheet" "" (id 3) (at 85.09 35.56 0)
+      (effects (font (size 1.27 1.27)) hide)
+    )
+    (property "UST_ID" "" (id 4) (at 85.09 35.56 0)
       (effects (font (size 1.27 1.27)) hide)
     )
@@
     (property "Reference" "C70" (id 0) (at 86.995 78.74 90))
     (property "Value" "100nF" (id 1) (at 89.535 87.63 90))
-    (property "Footprint" "Mlab_C:SMD-0603" (id 2) (at 84.7598 80.01 0)
-      (effects (font (size 1.27 1.27)) hide)
-    )
-    (property "Datasheet" "~" (id 3) (at 85.725 83.82 0)
-      (effects (font (size 1.27 1.27)) hide)
-    )
-    (property "UST_ID" "5c70984712875079b91f8b4c" (id 4) (at 85.725 83.82 0)
+    (property "Footprint" "Capacitor_SMD:C_0603_1608Metric" (id 2) (at 84.7598 80.01 0)
+      (effects (font (size 1.27 1.27)) hide)
+    )
+    (property "Datasheet" "" (id 3) (at 85.725 83.82 0)
+      (effects (font (size 1.27 1.27)) hide)
+    )
+    (property "UST_ID" "" (id 4) (at 85.725 83.82 0)
       (effects (font (size 1.27 1.27)) hide)
     )
@@
     (property "Reference" "C71" (id 0) (at 143.51 33.02 90))
     (property "Value" "100nF" (id 1) (at 144.78 30.48 90))
-    (property "Footprint" "Mlab_C:SMD-0603" (id 2) (at 135.89 30.1752 0)
-      (effects (font (size 1.27 1.27)) hide)
-    )
-    (property "Datasheet" "~" (id 3) (at 139.7 29.21 0)
-      (effects (font (size 1.27 1.27)) hide)
-    )
-    (property "UST_ID" "5c70984712875079b91f8b4c" (id 4) (at 139.7 29.21 0)
+    (property "Footprint" "Capacitor_SMD:C_0603_1608Metric" (id 2) (at 135.89 30.1752 0)
+      (effects (font (size 1.27 1.27)) hide)
+    )
+    (property "Datasheet" "" (id 3) (at 139.7 29.21 0)
+      (effects (font (size 1.27 1.27)) hide)
+    )
+    (property "UST_ID" "" (id 4) (at 139.7 29.21 0)
       (effects (font (size 1.27 1.27)) hide)
     )
@@
     (property "Reference" "C72" (id 0) (at 144.145 81.28 90))
     (property "Value" "100nF" (id 1) (at 145.415 78.74 90))
-    (property "Footprint" "Mlab_C:SMD-0603" (id 2) (at 136.525 78.4352 0)
-      (effects (font (size 1.27 1.27)) hide)
-    )
-    (property "Datasheet" "~" (id 3) (at 140.335 77.47 0)
-      (effects (font (size 1.27 1.27)) hide)
-    )
-    (property "UST_ID" "5c70984712875079b91f8b4c" (id 4) (at 140.335 77.47 0)
+    (property "Footprint" "Capacitor_SMD:C_0603_1608Metric" (id 2) (at 136.525 78.4352 0)
+      (effects (font (size 1.27 1.27)) hide)
+    )
+    (property "Datasheet" "" (id 3) (at 140.335 77.47 0)
+      (effects (font (size 1.27 1.27)) hide)
+    )
+    (property "UST_ID" "" (id 4) (at 140.335 77.47 0)
       (effects (font (size 1.27 1.27)) hide)
     )
@@
     (property "Reference" "C81" (id 0) (at 208.28 38.1 90))
     (property "Value" "100nF" (id 1) (at 213.36 33.655 90))
-    (property "Footprint" "Mlab_C:SMD-0603" (id 2) (at 208.5848 27.94 0)
-      (effects (font (size 1.27 1.27)) hide)
-    )
-    (property "Datasheet" "~" (id 3) (at 209.55 31.75 0)
-      (effects (font (size 1.27 1.27)) hide)
-    )
-    (property "UST_ID" "5c70984812875079b91f8bbe" (id 4) (at 209.55 31.75 0)
+    (property "Footprint" "Capacitor_SMD:C_0603_1608Metric" (id 2) (at 208.5848 27.94 0)
+      (effects (font (size 1.27 1.27)) hide)
+    )
+    (property "Datasheet" "" (id 3) (at 209.55 31.75 0)
+      (effects (font (size 1.27 1.27)) hide)
+    )
+    (property "UST_ID" "" (id 4) (at 209.55 31.75 0)
       (effects (font (size 1.27 1.27)) hide)
     )
@@
     (property "Reference" "C82" (id 0) (at 208.915 86.36 90))
     (property "Value" "100nF" (id 1) (at 213.995 81.915 90))
-    (property "Footprint" "Mlab_C:SMD-0603" (id 2) (at 209.2198 76.2 0)
-      (effects (font (size 1.27 1.27)) hide)
-    )
-    (property "Datasheet" "~" (id 3) (at 210.185 80.01 0)
-      (effects (font (size 1.27 1.27)) hide)
-    )
-    (property "UST_ID" "5c70984812875079b91f8bbe" (id 4) (at 210.185 80.01 0)
-      (effects (font (size 1.27 1.27)) hide)
-    )
+    (property "Footprint" "Capacitor_SMD:C_0603_1608Metric" (id 2) (at 209.2198 76.2 0)
+      (effects (font (size 1.27 1.27)) hide)
+    )
+    (property "Datasheet" "" (id 3) (at 210.185 80.01 0)
+      (effects (font (size 1.27 1.27)) hide)
+    )
+    (property "UST_ID" "" (id 4) (at 210.185 80.01 0)
+      (effects (font (size 1.27 1.27)) hide)
+    )

Commit message: Edit PCB
Parts:
- removed R43, R45: 100k, Resistor_SMD:R_0603_1608Metric, symbol Device:R
- removed R44, R46: -, Resistor_SMD:R_0603_1608Metric, symbol Device:R
- removed R49, R50: 0R, Resistor_SMD:R_0603_1608Metric, symbol Device:R
- L48, L49: value 1uH -> 1u5H - ETQ-P3M1R5KVP; footprint Mlab_L:DE1205-10 -> Mlab_L:PCC-M0530M-LP; UST_ID 5c70984412875079b91f8823 -> (none)
Connections:
- net VCC: now also U10.5 (EN), U11.5 (EN)
- net at U10.6 (VBST): now also C71.2
- net at C72.2: now also U11.6 (VBST)
