File: hw/sch_pcb/QFHMIX01D.kicad_sch (KiCad schematic)
At the start: 81 parts, among them J1 HEADER_1x08, J2 +9V, M1 HOLE, M2 HOLE, M3 HOLE, M4 HOLE, M5 HOLE, M6 HOLE, M7 HOLE, M8 HOLE, U12 Si53322, U2 AD8343, U3 AD8343, U5 LT6604-10

Commit message: Zmena pouzder L 0805.
Parts:
- C1, C12, C13, C19, C2, C20, C21, C22, C25, C26, C28, C8, C9: value 100nF -> (none); footprint Capacitor_SMD:C_0603_1608Metric -> (none)
- C10, C11, C15, C16, C17, C18, C23, C24, C3, C4, C5, C6, C7: value 10nF -> (none); footprint Capacitor_SMD:C_0603_1608Metric -> (none)
- C27: value 10uF/16 -> (none); footprint Capacitor_SMD:C_0805_2012Metric -> (none)
- D1: value M4 -> (none); footprint Diode_SMD:D_SMA -> (none)
- J1: value HEADER_1x08 -> (none); footprint Mlab_CON:IDC381-8-110 -> (none)
- J2: value +9V -> (none); footprint Mlab_Pin_Headers:Straight_2x03 -> (none)
- L1, L2, L3, L4: value 56nH -> (none); footprint Inductor_SMD:L_0805_2012Metric -> (none)
- L10, L13, L6, L9: value 270nH -> (none); footprint Inductor_SMD:L_0805_2012Metric -> (none)
- L11, L12, L7, L8: value 820nH -> (none); footprint Inductor_SMD:L_0805_2012Metric -> (none)
- M1, M2, M3, M4, M5, M6, M7, M8: value HOLE -> (none); footprint Mlab_Mechanical:MountingHole_3mm -> (none)
- R1, R2, R3, R4, R5, R6, R7, R8: value 68R -> (none); footprint Resistor_SMD:R_0603_1608Metric -> (none)
- R10, R9: value 3R9 -> (none); footprint Resistor_SMD:R_0603_1608Metric -> (none)
- R11, R13, R14, R15: value 130R -> (none); footprint Resistor_SMD:R_0603_1608Metric -> (none)
- R12, R27, R28, R29, R30: value 100R -> (none); footprint Resistor_SMD:R_0603_1608Metric -> (none)
- R23, R24, R25, R26: value 0R -> (none); footprint Resistor_SMD:R_0603_1608Metric -> (none)
- R31, R32, R33, R34: value 49R9 -> (none); footprint Resistor_SMD:R_0603_1608Metric -> (none)
- U12: value Si53322 -> (none); footprint Package_DFN_QFN:QFN-16-1EP_3x3mm_P0.5mm_EP1.7x1.7mm_ThermalVias -> (none)
- U2, U3: value AD8343 -> (none); footprint Package_SO:TSSOP-14_4.4x5mm_P0.65mm -> (none)
- U5: value LT6604-10 -> (none); footprint Mlab_IO:UFF_QFN34 -> (none)

Commit message: Add a link to clock buffer datasheet.
Parts:
- C1, C12, C13, C19, C2, C20, C21, C22, C25, C26, C28, C8, C9: value (none) -> 100nF; footprint (none) -> Capacitor_SMD:C_0603_1608Metric
- C10, C11, C15, C16, C17, C18, C23, C24, C3, C4, C5, C6, C7: value (none) -> 10nF; footprint (none) -> Capacitor_SMD:C_0603_1608Metric
- C27: value (none) -> 10uF/16; footprint (none) -> Capacitor_SMD:C_0805_2012Metric
- D1: value (none) -> M4; footprint (none) -> Diode_SMD:D_SMA
- J1: value (none) -> HEADER_1x08; footprint (none) -> Mlab_CON:IDC381-8-110
- J2: value (none) -> +9V; footprint (none) -> Mlab_Pin_Headers:Straight_2x03
- L1, L2, L3, L4: value (none) -> 56nH; footprint (none) -> Inductor_SMD:L_0805_2012Metric_Pad1.15x1.40mm_HandSolder
- L10, L13, L6, L9: value (none) -> 270nH; footprint (none) -> Inductor_SMD:L_0805_2012Metric_Pad1.15x1.40mm_HandSolder
- L11, L12, L7, L8: value (none) -> 820nH; footprint (none) -> Inductor_SMD:L_0805_2012Metric_Pad1.15x1.40mm_HandSolder
- M1, M2, M3, M4, M5, M6, M7, M8: value (none) -> HOLE; footprint (none) -> Mlab_Mechanical:MountingHole_3mm
- R1, R2, R3, R4, R5, R6, R7, R8: value (none) -> 68R; footprint (none) -> Resistor_SMD:R_0603_1608Metric
- R10, R9: value (none) -> 3R9; footprint (none) -> Resistor_SMD:R_0603_1608Metric
- R11, R13, R14, R15: value (none) -> 130R; footprint (none) -> Resistor_SMD:R_0603_1608Metric
- R12, R27, R28, R29, R30: value (none) -> 100R; footprint (none) -> Resistor_SMD:R_0603_1608Metric
- R23, R24, R25, R26: value (none) -> 0R; footprint (none) -> Resistor_SMD:R_0603_1608Metric
- R31, R32, R33, R34: value (none) -> 49R9; footprint (none) -> Resistor_SMD:R_0603_1608Metric
- U12: value (none) -> Si53322; footprint (none) -> Package_DFN_QFN:QFN-16-1EP_3x3mm_P0.5mm_EP1.7x1.7mm_ThermalVias
- U2, U3: value (none) -> AD8343; footprint (none) -> Package_SO:TSSOP-14_4.4x5mm_P0.65mm
- U5: value (none) -> LT6604-10; footprint (none) -> Mlab_IO:UFF_QFN34

Commit message: rozpracovani #11 (menic na 5 a 3v3)
Parts:
- renumbered C2 to C1, C4 to C10, C5 to C11, C6 to C12, C7 to C13, C15 to C14, C16 to C15, C17 to C16, C18 to C17, C19 to C18, C20 to C19, C1 to C2, C21 to C20, C22 to C21, C23 to C22, C24 to C23, C25 to C24, C26 to C25, C27 to C26, C28 to C27, C8 to C4, C9 to C5, C10 to C6, C11 to C7, C12 to C8, C13 to C9, L11 to L10, L12 to L11, L13 to L12, L6 to L5, L7 to L6, L8 to L7, L9 to L8, L10 to L9, M2 to M1, M1 to M2, R12 to R1, R4 to R10, R5 to R11, R9 to R12, R10 to R13, R7 to R14, R8 to R15, R23 to R16, R24 to R17, R25 to R18, R26 to R19, R1 to R2, R27 to R20, R28 to R21, R29 to R22, R30 to R23, R31 to R24, R32 to R25, R33 to R26, R34 to R27, R2 to R3, R3 to R4, R6 to R5, R11 to R6, R13 to R7, R14 to R8, R15 to R9, U12 to U1, U5 to U4

Commit message: Pridani novych otvoru pro sloupky pro montaz anteny #20, WIP
Parts:
- M1, M2, M3, M4: footprint Mlab_Mechanical:MountingHole_3mm -> Mlab_Mechanical:WA-SMSI_SMT_Steel_Spacer
