File: hw/sch_pcb/QFHMIX01E.kicad_sch (KiCad schematic)
At the start: 81 parts, among them J1 HEADER_1x08, J2 +9V, M1 HOLE, M2 HOLE, M3 HOLE, M4 HOLE, M5 HOLE, M6 HOLE, M7 HOLE, M8 HOLE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

Commit message: Renaming project to match name of new revision.
Other:
- title: QFHMIX01D -> QFHMIX01E
Changed lines of the file:
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@@
   (paper "A4")
   (title_block
-    (title "QFHMIX01D")
-    (date "2021-04-21")
+    (title "QFHMIX01E")
+    (date "2022-07-31")
     (comment 2 "Frontend for QFH active antenna")
   )
